Commit message: Changed simulation package name from 'watchdog' to simulation_watchdog'. Modified keyboard_controller package to not reset speed_lvl variable when stopping movement

File: simulation_watchdog/urdf/watchdog.urdf (robot description, URDF)
Before this commit: robot watchdog, 10 links, 9 joints
Links:
- link Battery_Link: geometry collision mesh filename=package://simulation_watchdog/meshes/Battery_Link.STL; visual mesh filename=package://simulation_watchdog/meshes/Battery_Link.STL
- link FreeWheel_Link: geometry collision mesh filename=package://simulation_watchdog/meshes/FreeWheel_Link.STL; visual mesh filename=package://simulation_watchdog/meshes/FreeWheel_Link.STL
- link LMotor_Link: geometry collision mesh filename=package://simulation_watchdog/meshes/LMotor_Link.STL; visual mesh filename=package://simulation_watchdog/meshes/LMotor_Link.STL
- link LWheel_Link: geometry collision mesh filename=package://simulation_watchdog/meshes/LWheel_Link.STL; visual mesh filename=package://simulation_watchdog/meshes/LWheel_Link.STL
- link Lidar_Link: geometry collision mesh filename=package://simulation_watchdog/meshes/Lidar_Link.STL; visual mesh filename=package://simulation_watchdog/meshes/Lidar_Link.STL
- link MotoShield_Link: geometry collision mesh filename=package://simulation_watchdog/meshes/MotoShield_Link.STL; visual mesh filename=package://simulation_watchdog/meshes/MotoShield_Link.STL
- link RMotor_Link: geometry collision mesh filename=package://simulation_watchdog/meshes/RMotor_Link.STL; visual mesh filename=package://simulation_watchdog/meshes/RMotor_Link.STL
- link RWheel_Link: geometry collision mesh filename=package://simulation_watchdog/meshes/RWheel_Link.STL; visual mesh filename=package://simulation_watchdog/meshes/RWheel_Link.STL
- link Rasp_Link: geometry collision mesh filename=package://simulation_watchdog/meshes/Rasp_Link.STL; visual mesh filename=package://simulation_watchdog/meshes/Rasp_Link.STL
- link base_link: geometry collision mesh filename=package://simulation_watchdog/meshes/base_link.STL; visual mesh filename=package://simulation_watchdog/meshes/base_link.STL

Commit message: Added new submodules, navigation and robot pose publisher. Fixed URDF files to have wheels be on the same side, added color to gazebo and rviz simulation.

File: simulation_watchdog/urdf/watchdog.urdf (robot description, URDF)
Before this commit: robot watchdog, 10 links, 9 joints
Links:
- removed link LMotor_Link
- removed link LWheel_Link
- removed link RMotor_Link
- removed link RWheel_Link
- added link LeMotor_Link, mass 0.0599050546017114; collision mesh filename=package://simulation_watchdog/meshes/LeMotor_Link.STL; visual mesh filename=package://simulation_watchdog/meshes/LeMotor_Link.STL
- added link LeWheel_Link, mass 0.15938; collision mesh filename=package://simulation_watchdog/meshes/LeWheel_Link.STL; visual mesh filename=package://simulation_watchdog/meshes/LeWheel_Link.STL
- added link RiMotor_Link, mass 0.0599050546017114; collision mesh filename=package://simulation_watchdog/meshes/RiMotor_Link.STL; visual mesh filename=package://simulation_watchdog/meshes/RiMotor_Link.STL
- added link RiWheel_Link, mass 0.15938; collision mesh filename=package://simulation_watchdog/meshes/RiWheel_Link.STL; visual mesh filename=package://simulation_watchdog/meshes/RiWheel_Link.STL
- link Lidar_Link: mass 0.0730824721228451 -> 0.0730824721237043
Joints:
- removed joint LMotor_Joint
- removed joint LWheel_Joint
- removed joint RMotor_Joint
- removed joint RWheel_Joint
- added joint LeMotor_Joint: type fixed, parent base_link, child LeMotor_Link, origin xyz=0.00306359051227961 0.0585 0.00629399818662646 rpy=-1.5707963267949 -1.11780647710814 0, axis 0 0 0
- added joint LeWheel_Joint: type continuous, parent base_link, child LeWheel_Link, origin xyz=0 0.089 0 rpy=1.5708 0 3.1416, axis 0 0 1
- added joint RiMotor_Joint: type fixed, parent base_link, child RiMotor_Link, origin xyz=0.00306359051226426 -0.0585 0.00629399818661908 rpy=1.5707963267949 0.452989849686705 0, axis 0 0 0
- added joint RiWheel_Joint: type continuous, parent base_link, child RiWheel_Link, origin xyz=0 -0.089 0 rpy=1.5708 0.74603 3.1416, axis 0 0 1
- joint FreeWheel_Joint: origin xyz=0.205365289585889 -0.000118819536407307 -0.0227799999999924 rpy=0 0 3.14159265358979 -> xyz=0.20537 -0.00011882 -0.02278 rpy=0 0 3.1416
- joint Rasp_Joint: origin xyz=0.215000000000015 0.05 0.0700000000000076 rpy=0 0 3.14159265358979 -> xyz=0.215 0.05 0.07 rpy=0 0 3.14159265358979
